Commit message: shadow Problem

File: src/robot_sim/urdf/robot.xacro (robot description, xacro)
@@ -131,4 +131,18 @@
     </collision>
   </link>
+<link name="camera_link">
+      <visual>
+        <origin xyz="0 0 0" rpy="0 0 0"/>
+        <geometry>
+      <box size="0.01 0.01 0.01"/>
+        </geometry>
+        <material name="orange"/>
+      </visual>
+      <inertial>
+        <mass value="1e-5" />
+        <origin xyz="0 0 0" rpy="0 0 0"/>
+        <inertia ixx="1e-6" ixy="0" ixz="0" iyy="1e-6" iyz="0" izz="1e-6" />
+      </inertial>
+</link>
 <joint    name="j2"    type="prismatic">
     <origin
@@ -143,4 +157,11 @@
       <limit effort="1000.0" lower="-0.23" upper="0.27" velocity="0.5"/>
   </joint>
+<joint name="camare_joints" type="prismatic">
+   <parent link="p2"/>
+   <child link="camera_link"/>
+   <limit effort="1000.0" lower="0.0" upper="0.0001" velocity="0.5"/>
+   <origin rpy="0 1.57 0" xyz="-0.02 -0.095 0"/>
+   <axis xyz="0 0 -1" />
+</joint>
 <!--bolbring -->
 <link    name="p3">
@@ -353,4 +374,93 @@
     </plugin>
 </gazebo>
+<gazebo reference="camera_link">
+  <sensor type="camera" name="camera1">
+    <update_rate>30.0</update_rate>
+    <camera name="head">
+      <horizontal_fov>1.3962634</horizontal_fov>
+      <image>
+        <width>800</width>
+        <height>800</height>
+        <format>R8G8B8</format>
+      </image>
+      <clip>
+        <near>0.02</near>
+        <far>300</far>
+      </clip>
+      <noise>
+        <type>gaussian</type>
+        <!-- Noise is sampled independently per pixel on each frame.
+             That pixel's noise value is added to each of its color
+             channels, which at that point lie in the range [0,1]. -->
+        <mean>0.0</mean>
+        <stddev>0.007</stddev>
+      </noise>
+    </camera>
+    <plugin name="camera_controller" filename="libgazebo_ros_camera.so">
+      <alwaysOn>true</alwaysOn>
+      <updateRate>0.0</updateRate>
+      <cameraName>rrbot/camera1</cameraName>
+      <imageTopicName>image_raw</imageTopicName>
+      <cameraInfoTopicName>camera_info</cameraInfoTopicName>
+      <frameName>camera_link</frameName>
+      <hackBaseline>0.07</hackBaseline>
+      <distortionK1>0.0</distortionK1>
+      <distortionK2>0.0</distortionK2>
+      <distortionK3>0.0</distortionK3>
+      <distortionT1>0.0</distortionT1>
+      <distortionT2>0.0</distortionT2>
+    </plugin>
+  </sensor>
+</gazebo>
+<gazebo reference="base_link">
+<collision name="base_link_collision">
+<surface>
+  <friction>
+    <ode>
+      <mu>100.0</mu>
+      <mu2>100.0</mu2>
+      <fdir1>0 0 0</fdir1>
+      <slip1>0</slip1>
+      <slip2>0</slip2>
+    </ode>
+    <torsional>
+      <coefficient>1</coefficient>
+      <patch_radius>0</patch_radius>
+      <surface_radius>0</surface_radius>
+      <use_patch_radius>1</use_patch_radius>
+      <ode>
+        <slip>0</slip>
+      </ode>
+    </torsional>
+  </friction>
+  <bounce>
+    <restitution_coefficient>0</restitution_coefficient>
+    <threshold>1e+06</threshold>
+  </bounce>
+  <contact>
+    <collide_without_contact>0</collide_without_contact>
+    <collide_without_contact_bitmask>1</collide_without_contact_bitmask>
+    <collide_bitmask>1</collide_bitmask>
+    <ode>
+      <soft_cfm>0</soft_cfm>
+      <soft_erp>0.2</soft_erp>
+      <kp>1e+13</kp>
+      <kd>1</kd>
+      <max_vel>0.01</max_vel>
+      <min_depth>0</min_depth>
+    </ode>
+    <bullet>
+      <split_impulse>1</split_impulse>
+      <split_impulse_penetration_threshold>-0.01</split_impulse_penetration_threshold>
+      <soft_cfm>0</soft_cfm>
+      <soft_erp>0.2</soft_erp>
+      <kp>1e+13</kp>
+      <kd>1</kd>
+    </bullet>
+  </contact>
+</surface>
+   </collision>
+    <material>Gazebo/White</material>
+</gazebo>
 <gazebo reference="p1">
     <material>Gazebo/Orange</material>
@@ -364,6 +474,100 @@
 <gazebo reference="p4">
     <material>Gazebo/Purple</material>
+    <collision name="p4_collision">
+    <surface>
+      <friction>
+        <ode>
+          <mu>100.0</mu>
+          <mu2>100.0</mu2>
+          <fdir1>0 0 0</fdir1>
+          <slip1>0</slip1>
+          <slip2>0</slip2>
+        </ode>
+        <torsional>
+          <coefficient>1</coefficient>
+          <patch_radius>0</patch_radius>
+          <surface_radius>0</surface_radius>
+          <use_patch_radius>1</use_patch_radius>
+          <ode>
+            <slip>0</slip>
+          </ode>
+        </torsional>
+      </friction>
+      <bounce>
+        <restitution_coefficient>0</restitution_coefficient>
+        <threshold>1e+06</threshold>
+      </bounce>
+      <contact>
+        <collide_without_contact>0</collide_without_contact>
+        <collide_without_contact_bitmask>1</collide_without_contact_bitmask>
+        <collide_bitmask>1</collide_bitmask>
+        <ode>
+          <soft_cfm>0</soft_cfm>
+          <soft_erp>0.2</soft_erp>
+          <kp>1e+13</kp>
+          <kd>1</kd>
+          <max_vel>0.01</max_vel>
+          <min_depth>0</min_depth>
+        </ode>
+        <bullet>
+          <split_impulse>1</split_impulse>
+          <split_impulse_penetration_threshold>-0.01</split_impulse_penetration_threshold>
+          <soft_cfm>0</soft_cfm>
+          <soft_erp>0.2</soft_erp>
+          <kp>1e+13</kp>
+          <kd>1</kd>
+        </bullet>
+      </contact>
+    </surface>
+       </collision>
 </gazebo>
 <gazebo reference="p5">
+<collision name="p5_collision">
+<surface>
+  <friction>
+    <ode>
+      <mu>100.0</mu>
+      <mu2>100.0</mu2>
+      <fdir1>0 0 0</fdir1>
+      <slip1>0</slip1>
+      <slip2>0</slip2>
+    </ode>
+    <torsional>
+      <coefficient>1</coefficient>
+      <patch_radius>0</patch_radius>
+      <surface_radius>0</surface_radius>
+      <use_patch_radius>1</use_patch_radius>
+      <ode>
+        <slip>0</slip>
+      </ode>
+    </torsional>
+  </friction>
+  <bounce>
+    <restitution_coefficient>0</restitution_coefficient>
+    <threshold>1e+06</threshold>
+  </bounce>
+  <contact>
+    <collide_without_contact>0</collide_without_contact>
+    <collide_without_contact_bitmask>1</collide_without_contact_bitmask>
+    <collide_bitmask>1</collide_bitmask>
+    <ode>
+      <soft_cfm>0</soft_cfm>
+      <soft_erp>0.2</soft_erp>
+      <kp>1e+13</kp>
+      <kd>1</kd>
+      <max_vel>0.01</max_vel>
+      <min_depth>0</min_depth>
+    </ode>
+    <bullet>
+      <split_impulse>1</split_impulse>
+      <split_impulse_penetration_threshold>-0.01</split_impulse_penetration_threshold>
+      <soft_cfm>0</soft_cfm>
+      <soft_erp>0.2</soft_erp>
+      <kp>1e+13</kp>
+      <kd>1</kd>
+    </bullet>
+  </contact>
+</surface>
+   </collision>
     <material>Gazebo/Red</material>
 </gazebo>

Commit message: modify world file

File: src/robot_sim/urdf/robot.xacro (robot description, xacro)
@@ -418,6 +418,6 @@
   <friction>
     <ode>
-      <mu>100.0</mu>
-      <mu2>100.0</mu2>
+      <mu>1.0</mu>
+      <mu2>1.0</mu2>
       <fdir1>0 0 0</fdir1>
       <slip1>0</slip1>
@@ -445,8 +445,8 @@
       <soft_cfm>0</soft_cfm>
       <soft_erp>0.2</soft_erp>
-      <kp>1e+13</kp>
+      <kp>1e+10</kp>
       <kd>1</kd>
-      <max_vel>0.01</max_vel>
-      <min_depth>0</min_depth>
+      <max_vel>0.1</max_vel>
+      <min_depth>0.001</min_depth>
     </ode>
     <bullet>
@@ -455,6 +455,6 @@
       <soft_cfm>0</soft_cfm>
       <soft_erp>0.2</soft_erp>
-      <kp>1e+13</kp>
-      <kd>1</kd>
+      <kp>1e+7</kp>
+      <kd>1.0</kd>
     </bullet>
   </contact>
@@ -464,69 +464,10 @@
 </gazebo>
 <gazebo reference="p1">
-    <material>Gazebo/Orange</material>
-</gazebo>
-<gazebo reference="p2">
-    <material>Gazebo/Blue</material>
-</gazebo>
-<gazebo reference="p3">
-    <material>Gazebo/Yellow</material>
-</gazebo>
-<gazebo reference="p4">
-    <material>Gazebo/Purple</material>
-    <collision name="p4_collision">
-    <surface>
-      <friction>
-        <ode>
-          <mu>100.0</mu>
-          <mu2>100.0</mu2>
-          <fdir1>0 0 0</fdir1>
-          <slip1>0</slip1>
-          <slip2>0</slip2>
-        </ode>
-        <torsional>
-          <coefficient>1</coefficient>
-          <patch_radius>0</patch_radius>
-          <surface_radius>0</surface_radius>
-          <use_patch_radius>1</use_patch_radius>
-          <ode>
-            <slip>0</slip>
-          </ode>
-        </torsional>
-      </friction>
-      <bounce>
-        <restitution_coefficient>0</restitution_coefficient>
-        <threshold>1e+06</threshold>
-      </bounce>
-      <contact>
-        <collide_without_contact>0</collide_without_contact>
-        <collide_without_contact_bitmask>1</collide_without_contact_bitmask>
-        <collide_bitmask>1</collide_bitmask>
-        <ode>
-          <soft_cfm>0</soft_cfm>
-          <soft_erp>0.2</soft_erp>
-          <kp>1e+13</kp>
-          <kd>1</kd>
-          <max_vel>0.01</max_vel>
-          <min_depth>0</min_depth>
-        </ode>
-        <bullet>
-          <split_impulse>1</split_impulse>
-          <split_impulse_penetration_threshold>-0.01</split_impulse_penetration_threshold>
-          <soft_cfm>0</soft_cfm>
-          <soft_erp>0.2</soft_erp>
-          <kp>1e+13</kp>
-          <kd>1</kd>
-        </bullet>
-      </contact>
-    </surface>
-       </collision>
-</gazebo>
-<gazebo reference="p5">
-<collision name="p5_collision">
+<collision name="p1_collision">
 <surface>
   <friction>
     <ode>
-      <mu>100.0</mu>
-      <mu2>100.0</mu2>
+      <mu>1.0</mu>
+      <mu2>1.0</mu2>
       <fdir1>0 0 0</fdir1>
       <slip1>0</slip1>
@@ -554,8 +495,8 @@
       <soft_cfm>0</soft_cfm>
       <soft_erp>0.2</soft_erp>
-      <kp>1e+13</kp>
+      <kp>1e+10</kp>
       <kd>1</kd>
-      <max_vel>0.01</max_vel>
-      <min_depth>0</min_depth>
+      <max_vel>0.1</max_vel>
+      <min_depth>0.001</min_depth>
     </ode>
     <bullet>
@@ -564,6 +505,206 @@
       <soft_cfm>0</soft_cfm>
       <soft_erp>0.2</soft_erp>
-      <kp>1e+13</kp>
+      <kp>1e+7</kp>
+      <kd>1.0</kd>
+    </bullet>
+  </contact>
+</surface>
+   </collision>
+    <material>Gazebo/Orange</material>
+</gazebo>
+<gazebo reference="p2">
+<collision name="p2_collision">
+<surface>
+  <friction>
+    <ode>
+      <mu>1.0</mu>
+      <mu2>1.0</mu2>
+      <fdir1>0 0 0</fdir1>
+      <slip1>0</slip1>
+      <slip2>0</slip2>
+    </ode>
+    <torsional>
+      <coefficient>1</coefficient>
+      <patch_radius>0</patch_radius>
+      <surface_radius>0</surface_radius>
+      <use_patch_radius>1</use_patch_radius>
+      <ode>
+        <slip>0</slip>
+      </ode>
+    </torsional>
+  </friction>
+  <bounce>
+    <restitution_coefficient>0</restitution_coefficient>
+    <threshold>1e+06</threshold>
+  </bounce>
+  <contact>
+    <collide_without_contact>0</collide_without_contact>
+    <collide_without_contact_bitmask>1</collide_without_contact_bitmask>
+    <collide_bitmask>1</collide_bitmask>
+    <ode>
+      <soft_cfm>0</soft_cfm>
+      <soft_erp>0.2</soft_erp>
+      <kp>1e+10</kp>
       <kd>1</kd>
+      <max_vel>0.1</max_vel>
+      <min_depth>0.001</min_depth>
+    </ode>
+    <bullet>
+      <split_impulse>1</split_impulse>
+      <split_impulse_penetration_threshold>-0.01</split_impulse_penetration_threshold>
+      <soft_cfm>0</soft_cfm>
+      <soft_erp>0.2</soft_erp>
+      <kp>1e+7</kp>
+      <kd>1.0</kd>
+    </bullet>
+  </contact>
+</surface>
+   </collision>
+    <material>Gazebo/Blue</material>
+</gazebo>
+<gazebo reference="p3">
+<collision name="p3_collision">
+<surface>
+  <friction>
+    <ode>
+      <mu>1.0</mu>
+      <mu2>1.0</mu2>
+      <fdir1>0 0 0</fdir1>
+      <slip1>0</slip1>
+      <slip2>0</slip2>
+    </ode>
+    <torsional>
+      <coefficient>1</coefficient>
+      <patch_radius>0</patch_radius>
+      <surface_radius>0</surface_radius>
+      <use_patch_radius>1</use_patch_radius>
+      <ode>
+        <slip>0</slip>
+      </ode>
+    </torsional>
+  </friction>
+  <bounce>
+    <restitution_coefficient>0</restitution_coefficient>
+    <threshold>1e+06</threshold>
+  </bounce>
+  <contact>
+    <collide_without_contact>0</collide_without_contact>
+    <collide_without_contact_bitmask>1</collide_without_contact_bitmask>
+    <collide_bitmask>1</collide_bitmask>
+    <ode>
+      <soft_cfm>0</soft_cfm>
+      <soft_erp>0.2</soft_erp>
+      <kp>1e+10</kp>
+      <kd>1</kd>
+      <max_vel>0.1</max_vel>
+      <min_depth>0.001</min_depth>
+    </ode>
+    <bullet>
+      <split_impulse>1</split_impulse>
+      <split_impulse_penetration_threshold>-0.01</split_impulse_penetration_threshold>
+      <soft_cfm>0</soft_cfm>
+      <soft_erp>0.2</soft_erp>
+      <kp>1e+7</kp>
+      <kd>1.0</kd>
+    </bullet>
+  </contact>
+</surface>
+   </collision>
+    <material>Gazebo/Yellow</material>
+</gazebo>
+<gazebo reference="p4">
+<collision name="p4_collision">
+<surface>
+  <friction>
+    <ode>
+      <mu>1.0</mu>
+      <mu2>1.0</mu2>
+      <fdir1>0 0 0</fdir1>
+      <slip1>0</slip1>
+      <slip2>0</slip2>
+    </ode>
+    <torsional>
+      <coefficient>1</coefficient>
+      <patch_radius>0</patch_radius>
+      <surface_radius>0</surface_radius>
+      <use_patch_radius>1</use_patch_radius>
+      <ode>
+        <slip>0</slip>
+      </ode>
+    </torsional>
+  </friction>
+  <bounce>
+    <restitution_coefficient>0</restitution_coefficient>
+    <threshold>1e+06</threshold>
+  </bounce>
+  <contact>
+    <collide_without_contact>0</collide_without_contact>
+    <collide_without_contact_bitmask>1</collide_without_contact_bitmask>
+    <collide_bitmask>1</collide_bitmask>
+    <ode>
+      <soft_cfm>0</soft_cfm>
+      <soft_erp>0.2</soft_erp>
+      <kp>1e+10</kp>
+      <kd>1</kd>
+      <max_vel>0.1</max_vel>
+      <min_depth>0.001</min_depth>
+    </ode>
+    <bullet>
+      <split_impulse>1</split_impulse>
+      <split_impulse_penetration_threshold>-0.01</split_impulse_penetration_threshold>
+      <soft_cfm>0</soft_cfm>
+      <soft_erp>0.2</soft_erp>
+      <kp>1e+7</kp>
+      <kd>1.0</kd>
+    </bullet>
+  </contact>
+</surface>
+   </collision>
+<material>Gazebo/Purple</material>
+</gazebo>
+<gazebo reference="p5">
+<collision name="p5_collision">
+<surface>
+  <friction>
+    <ode>
+      <mu>1.0</mu>
+      <mu2>1.0</mu2>
+      <fdir1>0 0 0</fdir1>
+      <slip1>0</slip1>
+      <slip2>0</slip2>
+    </ode>
+    <torsional>
+      <coefficient>1</coefficient>
+      <patch_radius>0</patch_radius>
+      <surface_radius>0</surface_radius>
+      <use_patch_radius>1</use_patch_radius>
+      <ode>
+        <slip>0</slip>
+      </ode>
+    </torsional>
+  </friction>
+  <bounce>
+    <restitution_coefficient>0</restitution_coefficient>
+    <threshold>1e+06</threshold>
+  </bounce>
+  <contact>
+    <collide_without_contact>0</collide_without_contact>
+    <collide_without_contact_bitmask>1</collide_without_contact_bitmask>
+    <collide_bitmask>1</collide_bitmask>
+    <ode>
+      <soft_cfm>0</soft_cfm>
+      <soft_erp>0.2</soft_erp>
+      <kp>1e+10</kp>
+      <kd>1</kd>
+      <max_vel>0.1</max_vel>
+      <min_depth>0.001</min_depth>
+    </ode>
+    <bullet>
+      <split_impulse>1</split_impulse>
+      <split_impulse_penetration_threshold>-0.01</split_impulse_penetration_threshold>
+      <soft_cfm>0</soft_cfm>
+      <soft_erp>0.2</soft_erp>
+      <kp>1e+7</kp>
+      <kd>1.0</kd>
     </bullet>
   </contact>
